File: Mps2762_Powersupply/_restore_backup_2026-07-26T05-01-04-238/Mps2762_Powersupply.kicad_sch (KiCad schematic)
At the start: 52 parts, among them J1 124018312112A, J2 Conn_01x08_Pin, J3 Conn_01x02_Pin, J4 Conn_01x02_Pin, SW1 SW_DIP_x03, U1 MP2762AGV-0000-P, U2 CH224K, U3 AP62600SJ-7

Commit message: partial layout complete
Connections:
- net PGND: no longer C2.2
- net SYS: no longer C2.1
Other:
- moved on the sheet: C14, C15
